File: hardware/v1.1/tiny-dap.kicad_pcb (KiCad board)
At the start: 2 copper layers, 25.4 x 10.2 mm, 15 parts, among them J1 USB_C_Receptacle_USB2.0, J2 Conn_02x04_Odd_Even, U1 MCU, U2 XC6206PxxxMR

Commit message: hardware bugfix.
- modify usb cc pin res val 22R -> 5K1.

Signed-off-by: UnsicentificLaLaLaLa <zhaohao1997@foxmail.com>
Parts:
- R1, R2: value 22R -> 5K1
Changed lines of the file:
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@@
         (effects (font (size 0.8 0.6) (thickness 0.15)))
     )
-    (fp_text value "22R" (at 0 1.43) (layer "F.Fab")
+    (fp_text value "5K1" (at 0 1.43) (layer "F.Fab")
         (effects (font (size 1 1) (thickness 0.15)))
     )
@@
         (effects (font (size 0.8 0.6) (thickness 0.15)))
     )
-    (fp_text value "22R" (at 0 1.43) (layer "F.Fab")
+    (fp_text value "5K1" (at 0 1.43) (layer "F.Fab")
         (effects (font (size 1 1) (thickness 0.15)))
     )
