File: hardware/v1.1/tiny-dap.kicad_sch (KiCad schematic)
At the start: 15 parts, among them J1 USB_C_Receptacle_USB2.0, J2 Conn_02x04_Odd_Even, U1 MCU, U2 XC6206PxxxMR

Commit message: hardware bugfix.
- modify usb cc pin res val 22R -> 5K1.

Signed-off-by: UnsicentificLaLaLaLa <zhaohao1997@foxmail.com>
Parts:
- R1, R2: value 22R -> 5K1
Changed lines of the file:
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@@
       (effects (font (size 1.27 1.27)))
     )
-    (property "Value" "22R" (at 232.41 55.88 90)
+    (property "Value" "5K1" (at 232.41 55.88 90)
       (effects (font (size 1.27 1.27)))
     )
@@
       (effects (font (size 1.27 1.27)))
     )
-    (property "Value" "22R" (at 232.41 53.34 90)
+    (property "Value" "5K1" (at 232.41 53.34 90)
       (effects (font (size 1.27 1.27)))
     )
